File: battery-buck-boost-dc-dc.kicad_pcb (KiCad board)
At the start: 2 copper layers, 15 x 12 mm, 9 parts, among them J1 Conn_01x03_Pin, U1 LTC3531EDD-TRPBF

Commit message: Remove JLC order number placeholder
Parts:
- moved QR 0.63 mm to (34.5, 31.4)
Other:
- board text removed: "JLCJLCJLCJLC"
Changed lines of the file:
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@@
 	(footprint "LOGO"
 		(layer "B.Cu")
-		(at 34.544 30.734 90)
+		(at 34.544 31.369 90)
 		(property "Reference" "QR"
 			(at 0 0 90)
@@
 		(layer "Edge.Cuts")
 	)
-	(gr_text "JLCJLCJLCJLC"
-		(at 34.544 36.195 0)
-		(layer "B.SilkS")
-		(effects
-			(font
-				(size 1 1)
-				(thickness 0.2)
-				(bold yes)
-			)
-			(justify mirror)
-		)
-	)
 	(dimension
