File: battery-buck-boost-dc-dc.kicad_sch (KiCad schematic)
At the start: 8 parts, among them J1 Conn_01x03_Pin, U1 LTC3531EDD-TRPBF

Commit message: Really fix resistor values
Parts:
- R1: value 442kΩ (3.3V) or 390kΩ (4V) or 374kΩ (4.5V) or 324kΩ (5V) 0.1% 125mW -> 590kΩ (3.3V) or 442kΩ (4V) or 374kΩ (4.5V) or 324kΩ (5V) 0.1% 125mW
Changed lines of the file:
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@@
 			)
 		)
-		(property "Value" "442kΩ (3.3V) or 390kΩ (4V) or 374kΩ (4.5V) or 324kΩ (5V) 0.1% 125mW"
+		(property "Value" "590kΩ (3.3V) or 442kΩ (4V) or 374kΩ (4.5V) or 324kΩ (5V) 0.1% 125mW"
 			(at 97.79 57.1499 0)
 			(effects
